Commit message: Refactor grip trajectory into 4 atomic phases and clean up parameter management
- Replace combined grip/laydown phases with 4 primitives: descend, close, open, lift
- Remove grip_z_offset from wall_plan_server, handle full offset in grip_traj_server
  (block_grip_z_offset + tcp_z_offset)
- Query world model for live block pickup poses with YAML fallback
- Publish virtual_tcp TF from grip_traj_server using tcp_z_offset (single source of truth)
- Rename gripper_open/close_angle to gripper_open/close_position (prismatic PZS100 rails)
- Add gripper_command_scale for sim/real parity (mimic joint doubles per-rail command)
- Visualize virtual TCP path in RViz instead of K8 path
- Add wall_plan_server.yaml config, accept wall_plans_file param
- Update rail joint limits to 0.7m for 1.4m total opening
- Remove dead __pycache__ dirs and empty orphaned directories

File: motion_planning/data/crane.urdf (robot description, URDF)
Before this commit: robot crane_model, 64 links, 63 joints
Joints:
- joint q11_right_rail_joint: limit lower=0 upper=0.538 effort=3.9e5 velocity=0.0995 -> lower=0 upper=0.7 effort=3.9e5 velocity=0.0995
- joint q9_left_rail_joint: limit lower=0 upper=0.538 effort=3.9e5 velocity=0.0995 -> lower=0 upper=0.7 effort=3.9e5 velocity=0.0995
